Commit message: jumping robot

File: Assignment5/data/body.urdf (robot description, URDF)
Before this commit: robot robot, 4 links, 3 joints
Links:
- removed link Crest
- removed link LeftWing
- removed link RightWing
- added link BackFoot, mass 1; collision box size=0.5 0.1 0.05; visual box size=0.5 0.1 0.05
- added link FrontFoot, mass 1; collision box size=0.5 0.1 0.05; visual box size=0.5 0.1 0.05
- added link LeftFoot, mass 1; collision box size=0.1 0.5 0.05; visual box size=0.1 0.5 0.05
- added link LowerLeg, mass 1; collision box size=0.1 0.1 0.4; visual box size=0.1 0.1 0.4
- added link RightFoot, mass 1; collision box size=0.1 0.5 0.05; visual box size=0.1 0.5 0.05
- added link UpperLeg, mass 1; collision box size=0.1 0.1 0.4; visual box size=0.1 0.1 0.4
- link Torso: geometry collision box size=0.3 0.3 0.3; visual box size=0.3 0.3 0.3
Joints:
- removed joint Torso_Crest
- removed joint Torso_LeftWing
- removed joint Torso_RightWing
- added joint LowerLeg_BackFoot: type revolute, parent LowerLeg, child BackFoot, origin xyz=0 0 -0.4 rpy=0 0 0, axis 0 1 0, limit lower=-3.14159 upper=3.14159 effort=0.0 velocity=0.0
- added joint LowerLeg_FrontFoot: type revolute, parent LowerLeg, child FrontFoot, origin xyz=0 0 -0.4 rpy=0 0 0, axis 0 1 0, limit lower=-3.14159 upper=3.14159 effort=0.0 velocity=0.0
- added joint LowerLeg_LeftFoot: type revolute, parent LowerLeg, child LeftFoot, origin xyz=0 0 -0.4 rpy=0 0 0, axis 1 0 0, limit lower=-3.14159 upper=3.14159 effort=0.0 velocity=0.0
- added joint LowerLeg_RightFoot: type revolute, parent LowerLeg, child RightFoot, origin xyz=0 0 -0.4 rpy=0 0 0, axis 1 0 0, limit lower=-3.14159 upper=3.14159 effort=0.0 velocity=0.0
- added joint Torso_UpperLeg: type revolute, parent Torso, child UpperLeg, origin xyz=0 0 0.8500000000000001 rpy=0 0 0, axis 0 1 0, limit lower=-3.14159 upper=3.14159 effort=0.0 velocity=0.0
- added joint UpperLeg_LowerLeg: type revolute, parent UpperLeg, child LowerLeg, origin xyz=0 0 -0.4 rpy=0 0 0, axis 0 1 0, limit lower=-3.14159 upper=3.14159 effort=0.0 velocity=0.0
